File: ECU_design/ECU.kicad_sch (KiCad schematic)
At the start: 34 parts, among them Q1 T23N03G, Q2 P9NK60ZFP, U1 Olimex_MOD-WIFI-ESP8266-DEV, U2 AMS1117-3.3, U3 MT3608_module, U4 LM324, U5 L7805

Commit message: improved 6v power input
Parts:
- U1: value Olimex_MOD-WIFI-ESP8266-DEV -> NodeMCU ESP8266; footprint Module:Olimex_MOD-WIFI-ESP8266-DEV -> (none)
Connections:
- net +6V_BATT: no longer U3.5 (IN)
- net 6V_CLEAN: now reaches L1.1, U2.3 (VI), ZD2.1 (K)
- net 6V_CLEAN: now also U3.5 (IN)
Other:
- note added: "Schmitt Trigger"
- moved on the sheet: C2, C4, D2, L1
